Commit message: added robot descriptor package and ROS2 devcontainers

File: src/freenove_description/urdf/robot.urdf (robot description, URDF)
Before this commit: robot big_hexapod, 25 links, 24 joints
Links:
- link base_link_2: geometry collision mesh filename=package://freenove_description/acoplecircular.stl; collision mesh filename=package://freenove_description/acoplecircular.stl
- link coxabl: geometry collision mesh filename=package://freenove_description/bigservo1.stl; collision mesh filename=package://freenove_description/bigservo1.stl
- link coxabr: geometry collision mesh filename=package://freenove_description/bigservo1.stl; collision mesh filename=package://freenove_description/bigservo1.stl
- link coxafl: geometry collision mesh filename=package://freenove_description/bigservo1.stl; collision mesh filename=package://freenove_description/bigservo1.stl
- link coxafr: geometry collision mesh filename=package://freenove_description/bigservo1.stl; collision mesh filename=package://freenove_description/bigservo1.stl
- link coxaml: geometry collision mesh filename=package://freenove_description/bigservo1.stl; collision mesh filename=package://freenove_description/bigservo1.stl
- link coxamr: geometry collision mesh filename=package://freenove_description/bigservo1.stl; collision mesh filename=package://freenove_description/bigservo1.stl
- link face: geometry collision mesh filename=package://freenove_description/camera.stl; collision mesh filename=package://freenove_description/faceplate.stl
- link femurbl: geometry collision mesh filename=package://freenove_description/acoplecircular.stl; collision mesh filename=package://freenove_description/acoplecircular.stl
- link femurbr: geometry collision mesh filename=package://freenove_description/acoplecircular.stl; collision mesh filename=package://freenove_description/acoplecircular.stl
- link femurfl: geometry collision mesh filename=package://freenove_description/acoplecircular.stl; collision mesh filename=package://freenove_description/acoplecircular.stl
- link femurfr: geometry collision mesh filename=package://freenove_description/acoplecircular.stl; collision mesh filename=package://freenove_description/acoplecircular.stl
- link femurml: geometry collision mesh filename=package://freenove_description/acoplecircular.stl; collision mesh filename=package://freenove_description/acoplecircular.stl
- link femurmr: geometry collision mesh filename=package://freenove_description/acoplecircular.stl; collision mesh filename=package://freenove_description/acoplecircular.stl
- link neck: geometry collision mesh filename=package://freenove_description/necksupport.stl; collision mesh filename=package://freenove_description/smallservo.stl
- link tibiabl: geometry collision mesh filename=package://freenove_description/bigservo1.stl; collision mesh filename=package://freenove_description/bigservo2.stl
- link tibiabr: geometry collision mesh filename=package://freenove_description/bigservo1.stl; collision mesh filename=package://freenove_description/bigservo2.stl
- link tibiafl: geometry collision mesh filename=package://freenove_description/bigservo1.stl; collision mesh filename=package://freenove_description/bigservo2.stl
- link tibiafr: geometry collision mesh filename=package://freenove_description/bigservo1.stl; collision mesh filename=package://freenove_description/bigservo2.stl
- link tibiaml: geometry collision mesh filename=package://freenove_description/bigservo1.stl; collision mesh filename=package://freenove_description/bigservo2.stl
- link tibiamr: geometry collision mesh filename=package://freenove_description/bigservo1.stl; collision mesh filename=package://freenove_description/bigservo2.stl

Commit message: fixed compilation errors, added friction and dampening to joints, fixed file links

File: src/freenove_description/urdf/robot.urdf (robot description, URDF)
Before this commit: robot big_hexapod, 25 links, 24 joints
Links:
- link base_link_2: geometry collision mesh filename=package://freenove_description/meshes/acoplecircular.stl; collision mesh filename=package://freenove_description/meshes/acoplecircular.stl
- link coxabl: geometry collision mesh filename=package://freenove_description/meshes/bigservo1.stl; collision mesh filename=package://freenove_description/meshes/bigservo1.stl
- link coxabr: geometry collision mesh filename=package://freenove_description/meshes/bigservo1.stl; collision mesh filename=package://freenove_description/meshes/bigservo1.stl
- link coxafl: geometry collision mesh filename=package://freenove_description/meshes/bigservo1.stl; collision mesh filename=package://freenove_description/meshes/bigservo1.stl
- link coxafr: geometry collision mesh filename=package://freenove_description/meshes/bigservo1.stl; collision mesh filename=package://freenove_description/meshes/bigservo1.stl
- link coxaml: geometry collision mesh filename=package://freenove_description/meshes/bigservo1.stl; collision mesh filename=package://freenove_description/meshes/bigservo1.stl
- link coxamr: geometry collision mesh filename=package://freenove_description/meshes/bigservo1.stl; collision mesh filename=package://freenove_description/meshes/bigservo1.stl
- link face: geometry collision mesh filename=package://freenove_description/meshes/camera.stl; collision mesh filename=package://freenove_description/meshes/faceplate.stl
- link femurbl: geometry collision mesh filename=package://freenove_description/meshes/acoplecircular.stl; collision mesh filename=package://freenove_description/meshes/acoplecircular.stl
- link femurbr: geometry collision mesh filename=package://freenove_description/meshes/acoplecircular.stl; collision mesh filename=package://freenove_description/meshes/acoplecircular.stl
- link femurfl: geometry collision mesh filename=package://freenove_description/meshes/acoplecircular.stl; collision mesh filename=package://freenove_description/meshes/acoplecircular.stl
- link femurfr: geometry collision mesh filename=package://freenove_description/meshes/acoplecircular.stl; collision mesh filename=package://freenove_description/meshes/acoplecircular.stl
- link femurml: geometry collision mesh filename=package://freenove_description/meshes/acoplecircular.stl; collision mesh filename=package://freenove_description/meshes/acoplecircular.stl
- link femurmr: geometry collision mesh filename=package://freenove_description/meshes/acoplecircular.stl; collision mesh filename=package://freenove_description/meshes/acoplecircular.stl
- link neck: geometry collision mesh filename=package://freenove_description/meshes/necksupport.stl; collision mesh filename=package://freenove_description/meshes/smallservo.stl
- link tibiabl: geometry collision mesh filename=package://freenove_description/meshes/bigservo1.stl; collision mesh filename=package://freenove_description/meshes/bigservo2.stl
- link tibiabr: geometry collision mesh filename=package://freenove_description/meshes/bigservo1.stl; collision mesh filename=package://freenove_description/meshes/bigservo2.stl
- link tibiafl: geometry collision mesh filename=package://freenove_description/meshes/bigservo1.stl; collision mesh filename=package://freenove_description/meshes/bigservo2.stl
- link tibiafr: geometry collision mesh filename=package://freenove_description/meshes/bigservo1.stl; collision mesh filename=package://freenove_description/meshes/bigservo2.stl
- link tibiaml: geometry collision mesh filename=package://freenove_description/meshes/bigservo1.stl; collision mesh filename=package://freenove_description/meshes/bigservo2.stl
- link tibiamr: geometry collision mesh filename=package://freenove_description/meshes/bigservo1.stl; collision mesh filename=package://freenove_description/meshes/bigservo2.stl
