Commit message: added sensor simulation

File: src/freenove_description/urdf/robot_gazebo.urdf (robot description, URDF)
Before this commit: robot big_hexapod, 25 links, 24 joints
Joints:
- joint camera_frame: origin xyz=0.0123472 -0.0288 0.0167 rpy=1.5708 -1.5708 0 -> xyz=0.0123472 -0.0288 0.0167 rpy=1.5708 0 -1.5708
- joint ultrasonic_frame: origin xyz=-0.012 -0.0301724 0.0297 rpy=1.5708 -1.5708 0 -> xyz=-0.012 -0.0301724 0.0297 rpy=1.5708 0 -1.5708
